File: stm32/Lily58.kicad_pcb (KiCad board)
At the start: 2 copper layers, 142.5 x 106.3 mm, 95 parts, among them J2 4PIN, J3 Conn_JTAG, J4 USB_C_Receptacle_USB2.0, P4 OLED, Q1 DTC123J, SW1 SW_PUSH, SW10 SW_PUSH, SW11 SW_PUSH, SW12 SW_PUSH, SW13 SW_PUSH, SW14 SW_PUSH, SW15 SW_PUSH, SW16 SW_PUSH, SW17 SW_PUSH, SW18 SW_PUSH, SW19 SW_PUSH, SW2 SW_PUSH, SW20 SW_PUSH, SW21 SW_PUSH, SW22 SW_PUSH, SW23 SW_PUSH, SW24 SW_PUSH, SW25 SW_PUSH, SW26 SW_PUSH, SW27 SW_PUSH, SW28 SW_PUSH, SW29 SW_PUSH, SW3 SW_PUSH, SW4 SW_PUSH, SW5 SW_PUSH, SW6 SW_PUSH, SW7 SW_PUSH, SW8 SW_PUSH, SW9 SW_PUSH, U1 STM32F072CBTx, U2 MCP23017_SO, U3 MCP1703A-3302_SOT23

Commit message: finishing pcb
Parts:
- C5, C6: value 0.1F -> 0.1uF; moved to B.Cu
- C9: value 10u -> 10uF
- J3: footprint Connector_PinSocket_2.54mm:PinSocket_1x04_P2.54mm_Horizontal -> Connector_PinSocket_2.54mm:PinSocket_1x04_P2.54mm_Vertical
- J4: footprint Connector_USB:USB_C_Receptacle_GCT_USB4085 -> Connector_USB:USB_C_Receptacle_Palconn_UTC16-G
- R3: moved to B.Cu
- moved C7 80.3 mm to (91.7, 79.2), turned to 90 degrees
- moved D30 77.6 mm to (89.8, 73.3), turned to 180 degrees
- moved C9 77.1 mm to (94.4, 69.8)
- moved C10 73.2 mm to (109.1, 53.0), turned to 270 degrees
- moved C1 65.3 mm to (102.3, 52.9), turned to 90 degrees
- moved C11 64.1 mm to (105.6, 53.1), turned to 270 degrees
- moved R3 63.2 mm to (103.4, 48.6)
- moved C3 62.6 mm to (98.9, 52.9), turned to 90 degrees
- moved C8 61.5 mm to (95.4, 79.2), turned to 90 degrees
- moved C5 57.6 mm to (98.9, 48.6), turned to 90 degrees
- moved C2 56.7 mm to (101.4, 71.0), turned to 270 degrees
- moved R6 55.4 mm to (94.3, 48.0), turned to 180 degrees
- moved R4 53.3 mm to (98.9, 48.3), turned to 270 degrees
- moved C4 52.8 mm to (89.9, 62.9), turned to 180 degrees
- moved C6 47.5 mm to (95.0, 48.6), turned to 90 degrees
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Connections:
- P4 pad 3: (no net) -> +3V3
- U1 pad 10: col0 -> (no net)
- U1 pad 11: col1 -> (no net)
- U1 pad 12: col2 -> row4
- U1 pad 13: col3 -> row3
- U1 pad 14: col4 -> row2
- U1 pad 16: (no net) -> row1
- U1 pad 17: (no net) -> row0
- U1 pad 18: row0 -> col4
- U1 pad 19: row1 -> col3
- U1 pad 20: row2 -> col2
- U1 pad 21: (no net) -> col1
- U1 pad 22: (no net) -> col0
- U1 pad 39: row3 -> (no net)
- U1 pad 40: row4 -> (no net)
- U1 pad 47: (no net) -> GND
- U2 pad 1: col0 -> row4
- U2 pad 2: col1 -> row3
- U2 pad 21: row4 -> col0
- U2 pad 22: row3 -> col1
- U2 pad 23: row2 -> col2
- U2 pad 24: row1 -> col3
- U2 pad 25: row0 -> col4
- U2 pad 26: (no net) -> row0
- U2 pad 3: col2 -> row2
- U2 pad 4: col3 -> col5
- U2 pad 5: col4 -> row1
- U2 pad 6: col5 -> (no net)
Routing:
- net +3V3: track 14.9 -> 155.5 mm, vias 0 -> 4
- net SCL: track 25.0 -> 75.5 mm, vias 1 -> 3
- net SWDIO: track 0.00 -> 45.1 mm, vias 0 -> 1
- net SWCLK: track 0.00 -> 43.3 mm, vias 0 -> 1
- net SDA: track 14.8 -> 51.3 mm, vias 1 -> 2
- net row4: track 126.4 -> 155.6 mm, vias 0 -> 1
- net D+: track 0.00 -> 27.8 mm
- net GND: track 6.01 -> 33.3 mm, vias 0 -> 11
- net VBUS: track 0.00 -> 25.9 mm
- net D-: track 0.00 -> 23.7 mm, vias 0 -> 2
- net NRST: track 0.00 -> 23.3 mm
- net row3: track 158.6 -> 181.9 mm, vias 0 -> 1
- net row2: track 138.8 -> 160.2 mm, vias 0 -> 1
- net col5: track 119.7 -> 140.6 mm, vias 0 -> 1
- net row1: track 129.5 -> 147.8 mm, vias 0 -> 1
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Other:
- board text added: "GND"
- board text added: "SWC"
- board text added: "SWD"
- board text added: "VCC"
