File: stm32/Lily58.sch (KiCad schematic (older format))
At the start: 95 parts, among them J2 4PIN, J3 Conn_JTAG, J4 USB_C_Receptacle_USB2.0, P4 OLED, Q1 DTC123J, SW1 SW_PUSH, SW10 SW_PUSH, SW11 SW_PUSH, SW12 SW_PUSH, SW13 SW_PUSH, SW14 SW_PUSH, SW15 SW_PUSH, SW16 SW_PUSH, SW17 SW_PUSH, SW18 SW_PUSH, SW19 SW_PUSH, SW2 SW_PUSH, SW20 SW_PUSH, SW21 SW_PUSH, SW22 SW_PUSH, SW23 SW_PUSH, SW24 SW_PUSH, SW25 SW_PUSH, SW26 SW_PUSH, SW27 SW_PUSH, SW28 SW_PUSH, SW29 SW_PUSH, SW3 SW_PUSH, SW4 SW_PUSH, SW5 SW_PUSH, SW6 SW_PUSH, SW7 SW_PUSH, SW8 SW_PUSH, SW9 SW_PUSH, U1 STM32F072CBTx, U2 MCP23017_SO, U3 MCP1703A-3302_SOT23

Commit message: finishing pcb
Parts:
- C5, C6: value 0.1F -> 0.1uF
- C9: value 10u -> 10uF
- J3: footprint Connector_PinSocket_2.54mm:PinSocket_1x04_P2.54mm_Horizontal -> Connector_PinSocket_2.54mm:PinSocket_1x04_P2.54mm_Vertical
- J4: footprint Connector_USB:USB_C_Receptacle_GCT_USB4085 -> Connector_USB:USB_C_Receptacle_Palconn_UTC16-G
Connections:
- net VCC is gone; now on net +3V3: P4.3 (P3)
- net GND: now also U1.47 (VSS)
- net col0: now also U1.22 (PB11), U2.21 (GPA0); no longer U1.10 (PA0), U2.1 (GPB0)
- net col1: now also U1.21 (PB10), U2.22 (GPA1); no longer U1.11 (PA1), U2.2 (GPB1)
- net col2: now also U1.20 (PB2), U2.23 (GPA2); no longer U1.12 (PA2), U2.3 (GPB2)
- net col3: now also U1.19 (PB1), U2.24 (GPA3); no longer U1.13 (PA3), U2.4 (GPB3)
- net col4: now also U1.18 (PB0), U2.25 (GPA4); no longer U1.14 (PA4), U2.5 (GPB4)
- net col5: now also U2.4 (GPB3); no longer U2.6 (GPB5)
- net row0: now also U1.17 (PA7), U2.26 (GPA5); no longer U1.18 (PB0), U2.25 (GPA4)
- net row1: now also U1.16 (PA6), U2.5 (GPB4); no longer U1.19 (PB1), U2.24 (GPA3)
- net row2: now also U1.14 (PA4), U2.3 (GPB2); no longer U1.20 (PB2), U2.23 (GPA2)
- net row3: now also U1.13 (PA3), U2.2 (GPB1); no longer U1.39 (PB3), U2.22 (GPA1)
- net row4: now also U1.12 (PA2), U2.1 (GPB0); no longer U1.40 (PB4), U2.21 (GPA0)
- no-connect marks 4 -> 32
Other:
- moved on the sheet: C5, C6, R3, U2
