File: atmega32u4/Lily58.sch (KiCad schematic (older format))
At the start: 96 parts, among them J2 4PIN, J4 USB_C_Receptacle_USB2.0, P4 OLED, SW1 SW_PUSH, SW10 SW_PUSH, SW11 SW_PUSH, SW12 SW_PUSH, SW13 SW_PUSH, SW14 SW_PUSH, SW15 SW_PUSH, SW16 SW_PUSH, SW17 SW_PUSH, SW18 SW_PUSH, SW19 SW_PUSH, SW2 SW_PUSH, SW20 SW_PUSH, SW21 SW_PUSH, SW22 SW_PUSH, SW23 SW_PUSH, SW24 SW_PUSH, SW25 SW_PUSH, SW26 SW_PUSH, SW27 SW_PUSH, SW28 SW_PUSH, SW29 SW_PUSH, SW3 SW_PUSH, SW4 SW_PUSH, SW5 SW_PUSH, SW6 SW_PUSH, SW7 SW_PUSH, SW8 SW_PUSH, SW9 SW_PUSH, U1 ATmega32U4-AU, U2 MCP23017_SO, U3 MCP1703A-3302_SOT23, Y1 16MHz

Commit message: removing ldo on atmega32u4
Parts:
- removed C10, C11: 1uF, Capacitor_SMD:C_0805_2012Metric, symbol Device:C
- removed U3: MCP1703A-3302_SOT23, Package_TO_SOT_SMD:SOT-23, symbol Regulator_Linear:MCP1703A-3302_SOT23
Connections:
- net +3V3: no longer C1.1, C2.1, C3.1, C4.1, C5.1, C6.1, J2.1, P4.3 (P3), R1.1, R2.1, R8.1, U1.14 (VCC), U1.2 (UVCC), U1.24 (AVCC), U1.34 (VCC), U1.44 (AVCC), U1.7 (VBUS), U2.9 (VDD)
- net +5V: now also C1.1, C2.1, C3.1, C4.1, C5.1, C6.1, J2.1, P4.3 (P3), R1.1, R2.1, R8.1, U1.14 (VCC), U1.2 (UVCC), U1.24 (AVCC), U1.34 (VCC), U1.44 (AVCC), U1.7 (VBUS), U2.9 (VDD)
Changed lines of the file:
@@
-$EndComp
-$Comp
-L Lily58-rescue:PWR_FLAG-Lily58-cache #FLG02
-U 1 1 5B74C9D1
-P 10950 4500
-F 0 "#FLG02" H 10950 4575 50  0001 C CNN
-F 1 "PWR_FLAG" H 10950 4673 50  0000 C CNN
-F 2 "" H 10950 4500 50  0001 C CNN
-F 3 "" H 10950 4500 50  0001 C CNN
-	1    10950 4500
-	-1   0    0    1
 $EndComp
 $Comp
@@
 SCL
 $Comp
-L Regulator_Linear:MCP1703A-3302_SOT23 U3
-U 1 1 6064AFB8
-P 8150 5600
-F 0 "U3" H 8150 5842 50  0000 C CNN
-F 1 "MCP1703A-3302_SOT23" H 8150 5751 50  0000 C CNN
-F 2 "Package_TO_SOT_SMD:SOT-23" H 8150 5800 50  0001 C CNN
-F 3 "http://ww1.microchip.com/downloads/en/DeviceDoc/20005122B.pdf" H 8150 5550 50  0001 C CNN
-	1    8150 5600
-	1    0    0    -1
-$EndComp
-$Comp
-L Device:C C11
-U 1 1 606533C4
-P 8650 5750
-F 0 "C11" H 8765 5796 50  0000 L CNN
-F 1 "1uF" H 8765 5705 50  0000 L CNN
-F 2 "Capacitor_SMD:C_0805_2012Metric" H 8688 5600 50  0001 C CNN
-F 3 "~" H 8650 5750 50  0001 C CNN
-	1    8650 5750
-	1    0    0    -1
-$EndComp
-$Comp
-L Device:C C10
-U 1 1 60653FE6
-P 7600 5750
-F 0 "C10" H 7715 5796 50  0000 L CNN
-F 1 "1uF" H 7715 5705 50  0000 L CNN
-F 2 "Capacitor_SMD:C_0805_2012Metric" H 7638 5600 50  0001 C CNN
-F 3 "~" H 7600 5750 50  0001 C CNN
-	1    7600 5750
-	1    0    0    -1
-$EndComp
-Connection ~ 8150 5900
-$Comp
-L power:GND #PWR0104
-U 1 1 6065CD72
-P 8150 6150
-F 0 "#PWR0104" H 8150 5900 50  0001 C CNN
-F 1 "GND" H 8155 5977 50  0000 C CNN
-F 2 "" H 8150 6150 50  0001 C CNN
-F 3 "" H 8150 6150 50  0001 C CNN
-	1    8150 6150
-	1    0    0    -1
-$EndComp
-Wire Wire Line
-	8150 5900 8150 6150
-$Comp
-L power:+3.3V #PWR0105
-U 1 1 6066FD9D
-P 8650 5400
-F 0 "#PWR0105" H 8650 5250 50  0001 C CNN
-F 1 "+3.3V" H 8665 5573 50  0000 C CNN
-F 2 "" H 8650 5400 50  0001 C CNN
-F 3 "" H 8650 5400 50  0001 C CNN
-	1    8650 5400
-	1    0    0    -1
-$EndComp
-$Comp
 L power:GND #PWR0106
 U 1 1 607182A0
@@
 	1    0    0    -1
 $EndComp
-Wire Wire Line
-	7600 5600 7850 5600
-Wire Wire Line
-	7600 5900 8150 5900
-Wire Wire Line
-	8450 5600 8650 5600
-Wire Wire Line
-	8650 5600 8650 5400
-Connection ~ 8650 5600
-Wire Wire Line
-	8150 5900 8650 5900
-Wire Wire Line
-	7600 5600 7600 5400
-Connection ~ 7600 5600
 $Comp
 L power:GND #PWR0111
@@
 Wire Wire Line
 	2700 10200 2700 10150
-$Comp
-L power:+3.3V #PWR0113
-U 1 1 60A9051E
-P 1200 6150
-F 0 "#PWR0113" H 1200 6000 50  0001 C CNN
-F 1 "+3.3V" H 1215 6323 50  0000 C CNN
-F 2 "" H 1200 6150 50  0001 C CNN
-F 3 "" H 1200 6150 50  0001 C CNN
-	1    1200 6150
-	1    0    0    -1
-$EndComp
 Wire Wire Line
 	1200 6150 1200 6300
@@
 Wire Wire Line
 	1650 5150 1950 5150
-$Comp
-L power:+3.3V #PWR0114
-U 1 1 60B0D7BC
-P 1950 4850
-F 0 "#PWR0114" H 1950 4700 50  0001 C CNN
-F 1 "+3.3V" H 1965 5023 50  0000 C CNN
-F 2 "" H 1950 4850 50  0001 C CNN
-F 3 "" H 1950 4850 50  0001 C CNN
-	1    1950 4850
-	1    0    0    -1
-$EndComp
 Wire Wire Line
 	1650 5050 1950 5050
 Wire Wire Line
 	1950 5050 1950 4850
-$Comp
-L power:+3.3V #PWR0119
-U 1 1 60C86A30
-P 10950 4500
-F 0 "#PWR0119" H 10950 4350 50  0001 C CNN
-F 1 "+3.3V" H 10965 4673 50  0000 C CNN
-F 2 "" H 10950 4500 50  0001 C CNN
-F 3 "" H 10950 4500 50  0001 C CNN
-	1    10950 4500
-	1    0    0    -1
-$EndComp
 Wire Wire Line
 	2500 6450 2700 6450
@@
 Wire Wire Line
 	2700 7650 2700 7950
-$Comp
-L power:+3.3V #PWR0123
-U 1 1 610513F7
-P 2700 7650
-F 0 "#PWR0123" H 2700 7500 50  0001 C CNN
-F 1 "+3.3V" H 2715 7823 50  0000 C CNN
-F 2 "" H 2700 7650 50  0001 C CNN
-F 3 "" H 2700 7650 50  0001 C CNN
-	1    2700 7650
-	1    0    0    -1
-$EndComp
 Wire Wire Line
 	5350 4200 5600 4200
@@
 	4600 3900 5100 3900
 Wire Wire Line
-	5350 3900 5600 3900
-Connection ~ 5350 3900
-Wire Wire Line
 	5600 3900 6050 3900
 Connection ~ 5600 3900
-Wire Wire Line
-	5100 3900 5350 3900
 $Comp
 L Device:C C4
@@
 $EndComp
 $Comp
-L power:+3.3V #PWR0125
-U 1 1 6092A8FD
-P 5350 3900
-F 0 "#PWR0125" H 5350 3750 50  0001 C CNN
-F 1 "+3.3V" H 5365 4073 50  0000 C CNN
-F 2 "" H 5350 3900 50  0001 C CNN
-F 3 "" H 5350 3900 50  0001 C CNN
-	1    5350 3900
-	1    0    0    -1
-$EndComp
-$Comp
 L power:GND #PWR0128
 U 1 1 61104BBC
@@
 NoConn ~ 2000 8850
 NoConn ~ 2000 8950
-$Comp
-L power:+3.3V #PWR0115
-U 1 1 6075752F
-P 2700 6350
-F 0 "#PWR0115" H 2700 6200 50  0001 C CNN
-F 1 "+3.3V" H 2715 6523 50  0000 C CNN
-F 2 "" H 2700 6350 50  0001 C CNN
-F 3 "" H 2700 6350 50  0001 C CNN
-	1    2700 6350
-	0    1    1    0
-$EndComp
 NoConn ~ 3400 8950
 NoConn ~ 3400 8850
@@
 Wire Wire Line
 	2000 10000 2000 9850
-Wire Wire Line
-	850  7450 1100 7450
 Wire Wire Line
 	850  7750 1100 7750
@@
 Wire Wire Line
 	1100 7750 1100 8050
-Wire Wire Line
-	1100 7450 1300 7450
-Connection ~ 1100 7450
 $Comp
 L Device:C C5
@@
 $EndComp
 $Comp
-L power:+3.3V #PWR0121
-U 1 1 609CDA7E
-P 1100 7450
-F 0 "#PWR0121" H 1100 7300 50  0001 C CNN
-F 1 "+3.3V" H 1115 7623 50  0000 C CNN
-F 2 "" H 1100 7450 50  0001 C CNN
-F 3 "" H 1100 7450 50  0001 C CNN
-	1    1100 7450
-	1    0    0    -1
-$EndComp
-$Comp
 L Interface_Expansion:MCP23017_SO U2
 U 1 1 605B56D2
@@
 Wire Wire Line
 	5000 5950 5100 5950
-$Comp
-L power:+5V #PWR0109
-U 1 1 608109C1
-P 7600 5400
-F 0 "#PWR0109" H 7600 5250 50  0001 C CNN
-F 1 "+5V" H 7615 5573 50  0000 C CNN
-F 2 "" H 7600 5400 50  0001 C CNN
-F 3 "" H 7600 5400 50  0001 C CNN
-	1    7600 5400
-	1    0    0    -1
-$EndComp
 $Comp
 L Lily58-rescue:PWR_FLAG-Lily58-cache #FLG0101
@@
 	1    0    0    -1
 $EndComp
-$Comp
-L power:+3.3V #PWR0101
-U 1 1 6063B683
-P 5000 5200
-F 0 "#PWR0101" H 5000 5050 50  0001 C CNN
-F 1 "+3.3V" H 5015 5373 50  0000 C CNN
-F 2 "" H 5000 5200 50  0001 C CNN
-F 3 "" H 5000 5200 50  0001 C CNN
-	1    5000 5200
-	1    0    0    -1
-$EndComp
 Wire Wire Line
 	5000 5350 5000 5200
@@
 Wire Wire Line
 	5700 5650 5800 5650
-$Comp
-L power:+3.3V #PWR0117
-U 1 1 607AB3F8
-P 5600 5400
-F 0 "#PWR0117" H 5600 5250 50  0001 C CNN
-F 1 "+3.3V" H 5615 5573 50  0000 C CNN
-F 2 "" H 5600 5400 50  0001 C CNN
-F 3 "" H 5600 5400 50  0001 C CNN
-	1    5600 5400
-	1    0    0    -1
-$EndComp
 Wire Wire Line
 	5600 5400 5600 5650
@@
 	4250 6650 4650 6650
 NoConn ~ 5100 6550
-$Comp
-L power:+3.3V #PWR0129
-U 1 1 607C95D3
+Wire Wire Line
+	4950 6750 5100 6750
+Wire Wire Line
+	850  7450 1100 7450
+Wire Wire Line
+	5100 3900 5350 3900
+$Comp
+L power:+5V #PWR0101
+U 1 1 60603B49
+P 5350 3900
+F 0 "#PWR0101" H 5350 3750 50  0001 C CNN
+F 1 "+5V" H 5365 4073 50  0000 C CNN
+F 2 "" H 5350 3900 50  0001 C CNN
+F 3 "" H 5350 3900 50  0001 C CNN
+	1    5350 3900
+	1    0    0    -1
+$EndComp
+Connection ~ 5350 3900
+Wire Wire Line
+	5350 3900 5600 3900
+$Comp
+L power:+5V #PWR0104
+U 1 1 60604A00
+P 5600 5400
+F 0 "#PWR0104" H 5600 5250 50  0001 C CNN
+F 1 "+5V" H 5615 5573 50  0000 C CNN
+F 2 "" H 5600 5400 50  0001 C CNN
+F 3 "" H 5600 5400 50  0001 C CNN
+	1    5600 5400
+	1    0    0    -1
+$EndComp
+$Comp
+L power:+5V #PWR0105
+U 1 1 6060590F
+P 5000 5200
+F 0 "#PWR0105" H 5000 5050 50  0001 C CNN
+F 1 "+5V" H 5015 5373 50  0000 C CNN
+F 2 "" H 5000 5200 50  0001 C CNN
+F 3 "" H 5000 5200 50  0001 C CNN
+	1    5000 5200
+	1    0    0    -1
+$EndComp
+$Comp
+L power:+5V #PWR0109
+U 1 1 6060663C
 P 4950 6750
-F 0 "#PWR0129" H 4950 6600 50  0001 C CNN
-F 1 "+3.3V" H 4965 6923 50  0000 C CNN
+F 0 "#PWR0109" H 4950 6600 50  0001 C CNN
+F 1 "+5V" H 4965 6923 50  0000 C CNN
 F 2 "" H 4950 6750 50  0001 C CNN
 F 3 "" H 4950 6750 50  0001 C CNN
@@
 	1    0    0    -1
 $EndComp
-Wire Wire Line
-	4950 6750 5100 6750
+$Comp
+L power:+5V #PWR0113
+U 1 1 606075A4
+P 1100 7450
+F 0 "#PWR0113" H 1100 7300 50  0001 C CNN
+F 1 "+5V" H 1115 7623 50  0000 C CNN
+F 2 "" H 1100 7450 50  0001 C CNN
+F 3 "" H 1100 7450 50  0001 C CNN
+	1    1100 7450
+	1    0    0    -1
+$EndComp
+Connection ~ 1100 7450
+Wire Wire Line
+	1100 7450 1300 7450
+$Comp
+L power:+5V #PWR0114
+U 1 1 6060B66F
+P 2700 7650
+F 0 "#PWR0114" H 2700 7500 50  0001 C CNN
+F 1 "+5V" H 2715 7823 50  0000 C CNN
+F 2 "" H 2700 7650 50  0001 C CNN
+F 3 "" H 2700 7650 50  0001 C CNN
+	1    2700 7650
+	1    0    0    -1
+$EndComp
+$Comp
+L power:+5V #PWR0115
+U 1 1 6061506D
+P 1200 6150
+F 0 "#PWR0115" H 1200 6000 50  0001 C CNN
+F 1 "+5V" H 1215 6323 50  0000 C CNN
+F 2 "" H 1200 6150 50  0001 C CNN
+F 3 "" H 1200 6150 50  0001 C CNN
+	1    1200 6150
+	1    0    0    -1
+$EndComp
+$Comp
+L power:+5V #PWR0117
+U 1 1 60615AE1
+P 2700 6350
+F 0 "#PWR0117" H 2700 6200 50  0001 C CNN
+F 1 "+5V" H 2715 6523 50  0000 C CNN
+F 2 "" H 2700 6350 50  0001 C CNN
+F 3 "" H 2700 6350 50  0001 C CNN
+	1    2700 6350
+	0    1    1    0
+$EndComp
+$Comp
+L power:+5V #PWR?
+U 1 1 60627093
+P 1950 4850
+F 0 "#PWR?" H 1950 4700 50  0001 C CNN
+F 1 "+5V" H 1965 5023 50  0000 C CNN
+F 2 "" H 1950 4850 50  0001 C CNN
+F 3 "" H 1950 4850 50  0001 C CNN
+	1    1950 4850
+	1    0    0    -1
+$EndComp
 $EndSCHEMATC
